File: design/electrical/UART_Adapter.sch (KiCad schematic (older format))
At the start: 15 parts, among them J1 DB9, P1 CONN_01X04, P2 CONN_01X04, U1 MAX3227

Commit message: Started PCB design
Parts:
- C1, C2, C3, C4, C5: footprint (none) -> Capacitors_SMD:C_0805_HandSoldering
- D1, D2, D3: footprint (none) -> LEDs:LED_0805
- J1: footprint (none) -> Connectors:DB9FC
- P1, P2: footprint (none) -> Socket_Strips:Socket_Strip_Straight_1x04
- R1, R2, R3: footprint (none) -> Resistors_SMD:R_0805_HandSoldering
- U1: footprint SSOP_Packages:SSOP-16_5.3x6.2mm_Pitch0.65mm -> Housings_SSOP:SSOP-16_5.3x6.2mm_Pitch0.65mm
Changed lines of the file:
@@
 F 0 "J1" H 2700 3000 50  0000 C CNN
 F 1 "DB9" H 2700 1900 50  0000 C CNN
-F 2 "" H 2700 2450 50  0000 C CNN
+F 2 "Connectors:DB9FC" H 2700 2450 50  0001 C CNN
 F 3 "" H 2700 2450 50  0000 C CNN
 	1    2700 2450
@@
 F 0 "D1" H 5250 2025 50  0000 L CNN
 F 1 "LED_Small" H 5125 1800 50  0000 L CNN
-F 2 "" V 5300 1900 50  0000 C CNN
+F 2 "LEDs:LED_0805" V 5300 1900 50  0001 C CNN
 F 3 "" V 5300 1900 50  0000 C CNN
 	1    5300 1900
@@
 F 0 "C1" H 4125 5850 50  0000 L CNN
 F 1 "0.1uF" H 4125 5650 50  0000 L CNN
-F 2 "" H 4138 5600 50  0000 C CNN
+F 2 "Capacitors_SMD:C_0805_HandSoldering" H 4138 5600 50  0001 C CNN
 F 3 "" H 4100 5750 50  0000 C CNN
 	1    4100 5750
@@
 F 0 "C2" H 3875 4100 50  0000 L CNN
 F 1 "0.1uF" H 3875 3900 50  0000 L CNN
-F 2 "" H 3888 3850 50  0000 C CNN
+F 2 "Capacitors_SMD:C_0805_HandSoldering" H 3888 3850 50  0001 C CNN
 F 3 "" H 3850 4000 50  0000 C CNN
 	1    3850 4000
@@
 F 0 "C3" H 6075 4100 50  0000 L CNN
 F 1 "0.1uF" H 6075 3900 50  0000 L CNN
-F 2 "" H 6088 3850 50  0000 C CNN
+F 2 "Capacitors_SMD:C_0805_HandSoldering" H 6088 3850 50  0001 C CNN
 F 3 "" H 6050 4000 50  0000 C CNN
 	1    6050 4000
@@
 F 0 "C4" H 6875 4600 50  0000 L CNN
 F 1 "0.1uF" H 6875 4400 50  0000 L CNN
-F 2 "" H 6888 4350 50  0000 C CNN
+F 2 "Capacitors_SMD:C_0805_HandSoldering" H 6888 4350 50  0001 C CNN
 F 3 "" H 6850 4500 50  0000 C CNN
 	1    6850 4500
@@
 F 0 "C5" H 6575 4900 50  0000 L CNN
 F 1 "0.1uF" H 6575 4700 50  0000 L CNN
-F 2 "" H 6588 4650 50  0000 C CNN
+F 2 "Capacitors_SMD:C_0805_HandSoldering" H 6588 4650 50  0001 C CNN
 F 3 "" H 6550 4800 50  0000 C CNN
 	1    6550 4800
@@
 F 0 "P1" H 7850 2250 50  0000 C CNN
 F 1 "CONN_01X04" V 7950 2000 50  0000 C CNN
-F 2 "" H 7850 2000 50  0000 C CNN
+F 2 "Socket_Strips:Socket_Strip_Straight_1x04" H 7850 2000 50  0001 C CNN
 F 3 "" H 7850 2000 50  0000 C CNN
 	1    7850 2000
@@
 F 0 "R1" V 5380 2200 50  0000 C CNN
 F 1 "1.5k" V 5300 2200 50  0000 C CNN
-F 2 "" V 5230 2200 50  0000 C CNN
+F 2 "Resistors_SMD:R_0805_HandSoldering" V 5230 2200 50  0001 C CNN
 F 3 "" H 5300 2200 50  0000 C CNN
 	1    5300 2200
@@
 F 0 "U1" H 4400 5800 50  0000 C CNN
 F 1 "MAX3227" H 5450 5800 50  0000 C CNN
-F 2 "SSOP_Packages:SSOP-16_5.3x6.2mm_Pitch0.65mm" H 4950 3450 50  0001 C CNN
+F 2 "Housings_SSOP:SSOP-16_5.3x6.2mm_Pitch0.65mm" H 4950 3450 50  0001 C CNN
 F 3 "" H 4950 4850 50  0000 C CNN
 	1    4950 4750
@@
 F 0 "P2" H 7850 2850 50  0000 C CNN
 F 1 "CONN_01X04" V 7950 2600 50  0000 C CNN
-F 2 "" H 7850 2600 50  0000 C CNN
+F 2 "Socket_Strips:Socket_Strip_Straight_1x04" H 7850 2600 50  0001 C CNN
 F 3 "" H 7850 2600 50  0000 C CNN
 	1    7850 2600
@@
 F 0 "D2" H 6000 5575 50  0000 L CNN
 F 1 "LED_Small" H 5875 5350 50  0000 L CNN
-F 2 "" V 6050 5450 50  0000 C CNN
+F 2 "LEDs:LED_0805" V 6050 5450 50  0001 C CNN
 F 3 "" V 6050 5450 50  0000 C CNN
 	1    6050 5450
@@
 F 0 "R2" V 6430 5450 50  0000 C CNN
 F 1 "1.5k" V 6350 5450 50  0000 C CNN
-F 2 "" V 6280 5450 50  0000 C CNN
+F 2 "Resistors_SMD:R_0805_HandSoldering" V 6280 5450 50  0001 C CNN
 F 3 "" H 6350 5450 50  0000 C CNN
 	1    6350 5450
@@
 F 0 "D3" H 5900 5975 50  0000 L CNN
 F 1 "LED_Small" H 5775 5750 50  0000 L CNN
-F 2 "" V 5950 5850 50  0000 C CNN
+F 2 "LEDs:LED_0805" V 5950 5850 50  0001 C CNN
 F 3 "" V 5950 5850 50  0000 C CNN
 	1    5950 5850
@@
 F 0 "R3" V 6030 6150 50  0000 C CNN
 F 1 "1.5k" V 5950 6150 50  0000 C CNN
-F 2 "" V 5880 6150 50  0000 C CNN
+F 2 "Resistors_SMD:R_0805_HandSoldering" V 5880 6150 50  0001 C CNN
 F 3 "" H 5950 6150 50  0000 C CNN
 	1    5950 6150
@@
 	4100 5950 4100 5900
 $Comp
-L PWR_FLAG #FLG?
+L PWR_FLAG #FLG014
 U 1 1 587904EB
 P 2450 4600
-F 0 "#FLG?" H 2450 4695 50  0001 C CNN
+F 0 "#FLG014" H 2450 4695 50  0001 C CNN
 F 1 "PWR_FLAG" H 2450 4780 50  0000 C CNN
 F 2 "" H 2450 4600 50  0000 C CNN
@@
 $EndComp
 $Comp
-L PWR_FLAG #FLG?
+L PWR_FLAG #FLG015
 U 1 1 5879051D
 P 2750 4750
-F 0 "#FLG?" H 2750 4845 50  0001 C CNN
+F 0 "#FLG015" H 2750 4845 50  0001 C CNN
 F 1 "PWR_FLAG" H 2750 4930 50  0000 C CNN
 F 2 "" H 2750 4750 50  0000 C CNN
@@
 $EndComp
 $Comp
-L GND #PWR?
+L GND #PWR016
 U 1 1 5879054F
 P 2450 4750
-F 0 "#PWR?" H 2450 4500 50  0001 C CNN
+F 0 "#PWR016" H 2450 4500 50  0001 C CNN
 F 1 "GND" H 2450 4600 50  0000 C CNN
 F 2 "" H 2450 4750 50  0000 C CNN
@@
 $EndComp
 $Comp
-L +3V3 #PWR?
+L +3V3 #PWR017
 U 1 1 58790581
 P 2750 4600
-F 0 "#PWR?" H 2750 4450 50  0001 C CNN
+F 0 "#PWR017" H 2750 4450 50  0001 C CNN
 F 1 "+3V3" H 2750 4740 50  0000 C CNN
 F 2 "" H 2750 4600 50  0000 C CNN
