File: design/electrical/uart_adapter.sch (KiCad schematic (older format))
At the start: 15 parts, among them J1 DB9, P1 CONN_01X04, P2 CONN_01X04, U1 MAX3227

Commit message: Added Molex connector
Parts:
- P1: footprint Socket_Strips:Socket_Strip_Straight_1x04 -> Connectors_Molex:Molex_PicoBlade_53261-0471_04x1.25mm_Angled
Changed lines of the file:
@@
 LIBS:contrib
 LIBS:valves
-LIBS:UART_Adapter-cache
+LIBS:uart_adapter-cache
 EELAYER 25 0
 EELAYER END
@@
 F 0 "P1" H 7850 2250 50  0000 C CNN
 F 1 "CONN_01X04" V 7950 2000 50  0000 C CNN
-F 2 "Socket_Strips:Socket_Strip_Straight_1x04" H 7850 2000 50  0001 C CNN
+F 2 "Connectors_Molex:Molex_PicoBlade_53261-0471_04x1.25mm_Angled" H 7850 2000 50  0001 C CNN
 F 3 "" H 7850 2000 50  0000 C CNN
 	1    7850 2000
