File: design/electrical/uart_adapter.kicad_pcb (KiCad board)
At the start: 2 copper layers, 33.2 x 44.8 mm, 15 parts, among them J1 DB9, P1 CONN_01X04, P2 CONN_01X04, U1 MAX3227

Commit message: Outline changed
Other:
- board size 33.2 x 44.8 mm -> 33.3 x 33.9 mm
Changed lines of the file:
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@@
     (links 32)
     (no_connects 0)
-    (area 132.576499 54.779499 165.937001 108.215501)
+    (area 132.512999 74.219999 166.000501 108.279001)
     (thickness 1.6)
-    (drawings 16)
+    (drawings 12)
     (tracks 114)
     (zones 0)
@@
   (layers
     (0 F.Cu signal)
-    (31 B.Cu signal hide)
+    (31 B.Cu signal)
     (32 B.Adhes user)
     (33 F.Adhes user)
@@
     (visible_elements 7FFFFFFF)
     (pcbplotparams
-      (layerselection 0x00030_80000001)
+      (layerselection 0x00020_80000001)
       (usegerberextensions false)
       (excludeedgelayer true)
@@
       (padsonsilk false)
       (subtractmaskfromsilk false)
-      (outputformat 1)
+      (outputformat 4)
       (mirror false)
-      (drillshape 1)
+      (drillshape 0)
       (scaleselection 1)
-      (outputdirectory ""))
+      (outputdirectory ../../production/electrical/))
   )
   (net 0 "")
@@
     )
   )
+  (gr_line (start 132.588 74.295) (end 165.9255 74.295) (angle 90) (layer Edge.Cuts) (width 0.15))
+  (gr_line (start 132.588 108.204) (end 132.588 74.295) (angle 90) (layer Edge.Cuts) (width 0.15))
+  (gr_line (start 165.9255 108.204) (end 132.588 108.204) (angle 90) (layer Edge.Cuts) (width 0.15))
+  (gr_line (start 165.9255 74.295) (end 165.9255 108.204) (angle 90) (layer Edge.Cuts) (width 0.15))
   (gr_text GND (at 160.8455 94.107 90) (layer F.SilkS)
     (effects (font (size 1.5 1.5) (thickness 0.3)))
   )
-  (gr_line (start 165.862 106.045) (end 165.862 108.1405) (angle 90) (layer Edge.Cuts) (width 0.15))
-  (gr_line (start 132.6515 108.1405) (end 132.969 108.1405) (angle 90) (layer Edge.Cuts) (width 0.15))
-  (gr_line (start 132.6515 106.045) (end 132.6515 108.1405) (angle 90) (layer Edge.Cuts) (width 0.15))
   (gr_text VAL (at 148.1455 101.5365) (layer F.SilkS)
     (effects (font (size 1.5 1.5) (thickness 0.3)))
@@
     (effects (font (size 1.5 1.5) (thickness 0.3)))
   )
-  (gr_line (start 132.969 63.373) (end 132.6515 63.373) (angle 90) (layer Edge.Cuts) (width 0.15))
-  (gr_line (start 132.969 63.373) (end 165.862 63.373) (angle 90) (layer Edge.Cuts) (width 0.15))
-  (gr_line (start 132.6515 106.045) (end 132.6515 63.373) (angle 90) (layer Edge.Cuts) (width 0.15))
-  (gr_line (start 165.862 108.1405) (end 132.969 108.1405) (angle 90) (layer Edge.Cuts) (width 0.15))
-  (gr_line (start 165.862 63.373) (end 165.862 106.045) (angle 90) (layer Edge.Cuts) (width 0.15))
   (segment (start 155.2785 87.955) (end 153.9315 87.955) (width 0.25) (layer F.Cu) (net 1))
   (segment (start 153.9315 87.955) (end 153.924 87.9475) (width 0.25) (layer F.Cu) (net 1))
@@
     (polygon
       (pts
-        (xy 132.715 63.4365) (xy 165.7985 63.4365) (xy 165.7985 108.077) (xy 132.715 108.077)
+        (xy 132.715 74.422) (xy 165.7985 74.422) (xy 165.7985 108.077) (xy 132.715 108.077)
       )
     )
@@
     (polygon
       (pts
-        (xy 132.715 63.4365) (xy 165.7985 63.4365) (xy 165.7985 108.077) (xy 132.715 108.077)
+        (xy 132.715 74.422) (xy 165.7985 74.422) (xy 165.7985 108.077) (xy 132.715 108.077)
       )
     )
